Commit message: fix files
Signed-off-by: Kenji Miyake <kenji.miyake@tier4.jp>

File: sample_vehicle_description/urdf/vehicle.xacro (robot description, xacro)
@@ -2,5 +2,5 @@
 <robot xmlns:xacro="http://ros.org/wiki/xacro">
   <!-- load parameter -->
-  <xacro:property name="vehicle_info" value="${load_yaml('$(find lexus_description)/config/vehicle_info.param.yaml')}"/>
+  <xacro:property name="vehicle_info" value="${load_yaml('$(find sample_vehicle_description)/config/vehicle_info.param.yaml')}"/>
   <!-- vehicle body -->
   <link name="base_link">
@@ -8,5 +8,5 @@
       <origin xyz="${vehicle_info['/**']['ros__parameters']['wheel_base']/2.0} 0 0" rpy="${pi/2.0} 0 ${pi}"/>
       <geometry>
-        <mesh filename="package://lexus_description/mesh/lexus.dae" scale="1 1 1"/>
+        <mesh filename="package://sample_vehicle_description/mesh/sample_vehicle.dae" scale="1 1 1"/>
       </geometry>
     </visual>

Commit message: ci(pre-commit): autofix

File: sample_vehicle_description/urdf/vehicle.xacro (robot description, xacro)
@@ -2,5 +2,8 @@
 <robot xmlns:xacro="http://ros.org/wiki/xacro">
   <!-- load parameter -->
-  <xacro:property name="vehicle_info" value="${load_yaml('$(find sample_vehicle_description)/config/vehicle_info.param.yaml')}"/>
+  <xacro:property
+    name="vehicle_info"
+    value="${load_yaml('$(find sample_vehicle_description)/config/vehicle_info.param.yaml')}"
+  />
   <!-- vehicle body -->
   <link name="base_link">
